Commit message: Removed mesh file prefix

File: assets/robots/hands/tesollo_hand/tesollo_hand_left.urdf (robot description, URDF)
Before this commit: robot delto_gripper_3f, 16 links, 15 joints
Links:
- link F1_01: geometry collision mesh filename=meshes/DG3F/link_01.stl; visual mesh filename=meshes/DG3F/link_01.stl
- link F1_02: geometry collision mesh filename=meshes/DG3F/link_02.stl; visual mesh filename=meshes/DG3F/link_02.stl
- link F1_03: geometry collision mesh filename=meshes/DG3F/link_03.stl; visual mesh filename=meshes/DG3F/link_03.stl
- link F1_04: geometry collision mesh filename=meshes/DG3F/link_04.stl; visual mesh filename=meshes/DG3F/link_04.stl
- link F1_TIP: geometry collision mesh filename=meshes/DG3F/link_tip_high.stl; visual mesh filename=meshes/DG3F/link_tip_high.stl
- link F2_01: geometry collision mesh filename=meshes/DG3F/link_01.stl; visual mesh filename=meshes/DG3F/link_01.stl
- link F2_02: geometry collision mesh filename=meshes/DG3F/link_02.stl; visual mesh filename=meshes/DG3F/link_02.stl
- link F2_03: geometry collision mesh filename=meshes/DG3F/link_03.stl; visual mesh filename=meshes/DG3F/link_03.stl
- link F2_04: geometry collision mesh filename=meshes/DG3F/link_04.stl; visual mesh filename=meshes/DG3F/link_04.stl
- link F2_TIP: geometry collision mesh filename=meshes/DG3F/link_tip_high.stl; visual mesh filename=meshes/DG3F/link_tip_high.stl
- link F3_01: geometry collision mesh filename=meshes/DG3F/link_01.stl; visual mesh filename=meshes/DG3F/link_01.stl
- link F3_02: geometry collision mesh filename=meshes/DG3F/link_02.stl; visual mesh filename=meshes/DG3F/link_02.stl
- link F3_03: geometry collision mesh filename=meshes/DG3F/link_03.stl; visual mesh filename=meshes/DG3F/link_03.stl
- link F3_04: geometry collision mesh filename=meshes/DG3F/link_04.stl; visual mesh filename=meshes/DG3F/link_04.stl
- link F3_TIP: geometry collision mesh filename=meshes/DG3F/link_tip_high.stl; visual mesh filename=meshes/DG3F/link_tip_high.stl
- link delto_base_link: geometry collision mesh filename=meshes/DG3F/delto_base_link.stl; visual mesh filename=meshes/DG3F/delto_base_link.stl

Commit message: Improved slightly by adding wrist joint

File: assets/robots/hands/tesollo_hand/tesollo_hand_left.urdf (robot description, URDF)
Before this commit: robot delto_gripper_3f, 16 links, 15 joints
Links:
- added link wrist
Joints:
- added joint wrist_joint: type fixed, parent delto_base_link, child wrist, origin xyz=0.0 -0.03 -0.05 rpy=0 0 -1.5708, axis 0.0 0.0 1.0
- joint F2M4: axis 0.0434 0.0 1.0 -> 0.0 0.0 1.0

Commit message: Added fingertips

File: assets/robots/hands/tesollo_hand/tesollo_hand_left.urdf (robot description, URDF)
Before this commit: robot delto_gripper_3f, 17 links, 16 joints
Links:
- added link F1_CONTACT
- added link F2_CONTACT
- added link F3_CONTACT
Joints:
- added joint CONTACT1: type fixed, parent F1_TIP, child F1_CONTACT, origin xyz=0.065 0.0 0.0 rpy=1.5708 0 1.5708
- added joint CONTACT2: type fixed, parent F2_TIP, child F2_CONTACT, origin xyz=0.065 0.0 0.0 rpy=1.5708 0 1.5708
- added joint CONTACT3: type fixed, parent F3_TIP, child F3_CONTACT, origin xyz=0.065 0.0 0.0 rpy=1.5708 0 1.5708
- joint wrist_joint: origin xyz=0.0 -0.03 -0.05 rpy=0 0 -1.5708 -> xyz=0.0 -0.03 0.02 rpy=0 -1.5708 -1.5708
