Commit message: Working on makeing teleoperation easier

File: dex_retarget/assets/robots/hands/tesollo_hand/tesollo_hand_right.urdf (robot description, URDF)
Before this commit: robot delto_gripper_3f, 20 links, 19 joints
Joints:
- joint CONTACT1: origin xyz=0.065 0.0 0.0 rpy=1.5708 0 1.5708 -> xyz=0.065 0.0 0.0 rpy=-1.57 0 0
